File: oscar_pcb_svg2shenzen.kicad_pcb (KiCad board)
At the start: 2 copper layers, 35.3 x 44.9 mm, 8 parts

Commit message: fix-logo
Parts:
- removed the G*** at (62.2, 58.4) (x7)
- added G*** (x7): LOGO, LOGO, F.Cu at (0.00, 0.00)
- moved ? 85.4 mm to (-1.80, -31.2)
